File: ChipChat_Project/BME280_Sheet.kicad_sch (KiCad schematic)
At the start: 1 part, among them U1 BME280

Commit message: 💾 snapshot 2025-12-30_22-11-59
Parts:
- removed U1: BME280, symbol Sensor:BME280
- added U1: MCP2210-I_SO, symbol MCP2210-I_SO
Changed lines of the file:
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@@
 	(paper "A4")
 	(symbol
-		(lib_id "Sensor:BME280")
+		(lib_id "MCP2210-I_SO")
 		(at 148.5 105.0 0)
 		(property "Reference" "U1"
@@
 			(effects (font (size 1.27 1.27)))
 		)
-		(property "Value" "BME280"
+		(property "Value" "MCP2210-I_SO"
 			(at 148.5 102.46 0)
 			(effects (font (size 1.27 1.27)))
