File: ChipChat_Project/ChipChat_Project.kicad_sch (KiCad schematic)
At the start: 0 parts

Commit message: 💾 snapshot 2025-12-30_22-45-14
Other:
- sheet BME280_Sheet renamed BME280_Sensor
- added sheet MCP2210_USB_TO_SPI (MCP2210_USB_TO_SPI.kicad_sch)
- sheet BME280_Sensor: file BME280_Sheet.kicad_sch -> BME280_Sensor.kicad_sch
Changed lines of the file:
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@@
 		(at 30.48 30.48)
 		(size 40.64 20.32)
-		(exclude_from_sim no)
-		(in_bom yes)
-		(on_board yes)
-		(dnp no)
-		(fields_autoplaced yes)
-		(stroke
-			(width 0.1524)
-			(type solid)
-		)
-		(fill
-			(color 0 0 0 0.0)
-		)
-		(property "Sheetname" "BME280_Sheet"
+		(property "Sheetname" "BME280_Sensor"
 			(at 30.48 29.8 0)
 			(effects (font (size 1.27 1.27)) (justify left bottom))
 		)
-		(property "Sheetfile" "BME280_Sheet.kicad_sch"
+		(property "Sheetfile" "BME280_Sensor.kicad_sch"
 			(at 30.48 51.0 0)
 			(effects (font (size 1.27 1.27)) (justify left top))
 		)
+	)
+    (sheet
+		(at 30.48 60.96)
+		(size 40.64 20.32)
+		(property "Sheetname" "MCP2210_USB_TO_SPI"
+			(at 30.48 59.6 0)
+			(effects (font (size 1.27 1.27)) (justify left bottom))
+		)
+		(property "Sheetfile" "MCP2210_USB_TO_SPI.kicad_sch"
+			(at 30.48 81.5 0)
+			(effects (font (size 1.27 1.27)) (justify left top))
+		)
