File: ChipChat_Project/BME280_Sensor.kicad_sch (KiCad schematic)
At the start: 1 part, among them U1 BME280

Commit message: 💾 snapshot 2025-12-30_23-52-56
Parts:
- U1: footprint BME280.kicad_mod -> Footprint_Library:BME280
Changed lines of the file:
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@@
 		(property "Reference" "U1" (at 148.5 107.54 0) (effects (font (size 1.27 1.27))))
 		(property "Value" "BME280" (at 148.5 102.46 0) (effects (font (size 1.27 1.27))))
-		(property "Footprint" "BME280.kicad_mod" (at 148.5 105.0 0) (effects (font (size 1.27 1.27)) (hide yes)))
+		(property "Footprint" "Footprint_Library:BME280" (at 148.5 105.0 0) (effects (font (size 1.27 1.27)) (hide yes)))
 		(property "Datasheet" "" (at 148.5 105.0 0) (effects (font (size 1.27 1.27)) (hide yes)))
 	)
