File: ChipChat_Project/MCP2210_USB_TO_SPI.kicad_sch (KiCad schematic)
At the start: 1 part, among them U1 MCP2210-I/SO

Commit message: 💾 snapshot 2025-12-30_23-52-56
Parts:
- U1: footprint MCP2210-I_SO.kicad_mod -> Footprint_Library:MCP2210-I_SO
Changed lines of the file:
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@@
 		(property "Reference" "U1" (at 148.5 107.54 0) (effects (font (size 1.27 1.27))))
 		(property "Value" "MCP2210-I/SO" (at 148.5 102.46 0) (effects (font (size 1.27 1.27))))
-		(property "Footprint" "MCP2210-I_SO.kicad_mod" (at 148.5 105.0 0) (effects (font (size 1.27 1.27)) (hide yes)))
+		(property "Footprint" "Footprint_Library:MCP2210-I_SO" (at 148.5 105.0 0) (effects (font (size 1.27 1.27)) (hide yes)))
 		(property "Datasheet" "" (at 148.5 105.0 0) (effects (font (size 1.27 1.27)) (hide yes)))
 	)
