File: ChipChat_Project/generated/BME280_Sensor.kicad_sch (KiCad schematic)
At the start: 1 part, among them U1 BME280

Commit message: 💾 snapshot 2026-02-22_23-42-09
Parts:
- removed U1: BME280, Footprint_Library:BME280, symbol BME280
- added C10, C9: 0.1uF, symbol Capacitor
- added R5, R6: 4.7K, symbol Resistor
- added R7, R8, R9: 0R, symbol Resistor
- added U3: BME280, symbol BME280
Connections:
- net GND: now also C10.1, C9.1, R9.1, U3.1 (GND), U3.7 (GND)
- new net I2C_SCL_0R: R7.1, U3.4 (SCK)
- new net I2C_SCL_BME: R5.2, R7.2
- new net I2C_SDA_0R: R8.1, U3.3 (SDI)
- new net I2C_SDA_BME: R6.2, R8.2
- new net PP_3V3_OUT: C10.2, C9.2, R5.1, R6.1, U3.6 (VDDIO), U3.8 (VDD)
- new net SDO_ADD: R9.2, U3.5 (SDO)
