File: ChipChat_Project/generated/library_test/library_test.kicad_sch (KiCad schematic)
At the start: 3 parts, among them U1 NE555D, U2 STM32F103C8Tx, U3 BME280

Commit message: 💾 snapshot 2026-03-18_12-00-13
Parts:
- removed U2: STM32F103C8Tx, symbol STM32F103C8Tx
- removed U3: BME280, symbol BME280
- added C1: 100nF, symbol Capacitor
- added U2: AP1117-15, symbol AP1117-15
- added U3: nRF5340-QKxx, symbol nRF5340-QKxx
- added U4: BME280, symbol BME280
- added U5: Resistor, symbol Resistor
Connections:
- net GND: now also U4.1 (GND), U4.7 (GND)
- new net: U3.A19 (VDD), U3.AC1 (VDD), U3.AG1 (VDD), U3.AJ31 (VDD), U3.AL11 (VDD), U3.AL17 (VDD), U3.AL25 (VDD), U3.AL3 (VDD), U3.AL7 (VDD), U3.B28 (VDD), U3.B8 (VDD), U3.C1 (VDD), U3.E31 (VDD), U3.L1 (VDD), U3.N31 (VDD), U3.U1 (VDD)
Changed lines of the file:
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@@
 	(symbol
 		(lib_id "NE555D")
-		(at 100.0 60.0 0)
-		(property "Reference" "U1" (at 100.0 62.54 0) (effects (font (size 1.27 1.27))))
-		(property "Value" "NE555D" (at 100.0 57.46 0) (effects (font (size 1.27 1.27))))
-		(property "Footprint" "" (at 100.0 60.0 0) (effects (font (size 1.27 1.27)) (hide yes)))
-		(property "Datasheet" "" (at 100.0 60.0 0) (effects (font (size 1.27 1.27)) (hide yes)))
+		(at 120.0 50.0 0)
+		(property "Reference" "U1" (at 120.0 52.54 0) (effects (font (size 1.27 1.27))))
+		(property "Value" "NE555D" (at 120.0 47.46 0) (effects (font (size 1.27 1.27))))
+		(property "Footprint" "" (at 120.0 50.0 0) (effects (font (size 1.27 1.27)) (hide yes)))
+		(property "Datasheet" "" (at 120.0 50.0 0) (effects (font (size 1.27 1.27)) (hide yes)))
 	)
 	(symbol
-		(lib_id "STM32F103C8Tx")
-		(at 100.0 140.0 0)
-		(property "Reference" "U2" (at 100.0 142.54 0) (effects (font (size 1.27 1.27))))
-		(property "Value" "STM32F103C8Tx" (at 100.0 137.46 0) (effects (font (size 1.27 1.27))))
-		(property "Footprint" "" (at 100.0 140.0 0) (effects (font (size 1.27 1.27)) (hide yes)))
-		(property "Datasheet" "" (at 100.0 140.0 0) (effects (font (size 1.27 1.27)) (hide yes)))
+		(lib_id "AP1117-15")
+		(at 120.0 120.0 0)
+		(property "Reference" "U2" (at 120.0 122.54 0) (effects (font (size 1.27 1.27))))
+		(property "Value" "AP1117-15" (at 120.0 117.46 0) (effects (font (size 1.27 1.27))))
+		(property "Footprint" "" (at 120.0 120.0 0) (effects (font (size 1.27 1.27)) (hide yes)))
+		(property "Datasheet" "" (at 120.0 120.0 0) (effects (font (size 1.27 1.27)) (hide yes)))
+	)
+	(symbol
+		(lib_id "nRF5340-QKxx")
+		(at 120.0 190.0 0)
+		(property "Reference" "U3" (at 120.0 192.54 0) (effects (font (size 1.27 1.27))))
+		(property "Value" "nRF5340-QKxx" (at 120.0 187.46 0) (effects (font (size 1.27 1.27))))
+		(property "Footprint" "" (at 120.0 190.0 0) (effects (font (size 1.27 1.27)) (hide yes)))
+		(property "Datasheet" "" (at 120.0 190.0 0) (effects (font (size 1.27 1.27)) (hide yes)))
 	)
 	(symbol
 		(lib_id "BME280")
-		(at 100.0 220.0 0)
-		(property "Reference" "U3" (at 100.0 222.54 0) (effects (font (size 1.27 1.27))))
-		(property "Value" "BME280" (at 100.0 217.46 0) (effects (font (size 1.27 1.27))))
-		(property "Footprint" "" (at 100.0 220.0 0) (effects (font (size 1.27 1.27)) (hide yes)))
-		(property "Datasheet" "" (at 100.0 220.0 0) (effects (font (size 1.27 1.27)) (hide yes)))
+		(at 120.0 260.0 0)
+		(property "Reference" "U4" (at 120.0 262.54 0) (effects (font (size 1.27 1.27))))
+		(property "Value" "BME280" (at 120.0 257.46 0) (effects (font (size 1.27 1.27))))
+		(property "Footprint" "" (at 120.0 260.0 0) (effects (font (size 1.27 1.27)) (hide yes)))
+		(property "Datasheet" "" (at 120.0 260.0 0) (effects (font (size 1.27 1.27)) (hide yes)))
+	)
+	(symbol
+		(lib_id "Resistor")
+		(at 120.0 330.0 0)
+		(property "Reference" "U5" (at 120.0 332.54 0) (effects (font (size 1.27 1.27))))
+		(property "Value" "Resistor" (at 120.0 327.46 0) (effects (font (size 1.27 1.27))))
+		(property "Footprint" "" (at 120.0 330.0 0) (effects (font (size 1.27 1.27)) (hide yes)))
+		(property "Datasheet" "" (at 120.0 330.0 0) (effects (font (size 1.27 1.27)) (hide yes)))
+	)
+	(symbol
+		(lib_id "Capacitor")
+		(at 120.0 400.0 0)
+		(property "Reference" "C1" (at 120.0 402.54 0) (effects (font (size 1.27 1.27))))
+		(property "Value" "100nF" (at 120.0 397.46 0) (effects (font (size 1.27 1.27))))
+		(property "Footprint" "" (at 120.0 400.0 0) (effects (font (size 1.27 1.27)) (hide yes)))
+		(property "Datasheet" "" (at 120.0 400.0 0) (effects (font (size 1.27 1.27)) (hide yes)))
 	)
 )
