File: ChipChat_Project/generated/LED_Blink_Project/LED_Blink_Project-backups/LED_Blink_Project-2026-03-18_122450/LED_Blink_Circuit.kicad_sch (KiCad schematic)
At the start: 6 parts, among them J1 Connector_Generic:Conn_01x02, J2 Connector_Generic:Conn_01x02, Q1 Transistor_FET:BS170

Commit message: 💾 snapshot 2026-03-18_12-44-45
Parts:
- removed LED1: LED_TH:LED_D5.0mm, symbol LED
- removed Q1: Transistor_FET:BS170, symbol Q_NMOS_GDS
- added LED1: LED_TH:LED_D5.0mm, symbol L
- added Q1: Transistor_FET:BS170, symbol BS170
Connections:
- net FET_DRAIN: now also LED1.2
- net LED_DRIVE: now also LED1.1
Changed lines of the file:
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@@
 	)
 	(symbol
-		(lib_id "LED")
+		(lib_id "L")
 		(at 220.0 100.0 0)
 		(unit 1)
@@
 	(wire
 		(pts
-			(xy 223.81 100.0) (xy 231.43 100.0)
+			(xy 220.0 96.19) (xy 220.0 86.03)
 		)
 		(stroke
@@
 	)
 	(label "LED_DRIVE"
-		(at 231.43 100.0 0)
+		(at 220.0 86.03 90)
 		(effects
 			(font
@@
 	(wire
 		(pts
-			(xy 216.19 100.0) (xy 208.57 100.0)
+			(xy 220.0 103.81) (xy 220.0 113.97)
 		)
 		(stroke
@@
 	)
 	(label "FET_DRAIN"
-		(at 208.57 100.0 0)
+		(at 220.0 113.97 90)
 		(effects
 			(font
@@
 	)
 	(symbol
-		(lib_id "Q_NMOS_GDS")
+		(lib_id "BS170")
 		(at 260.0 100.0 0)
 		(unit 1)
@@
 		)
 	)
-	(wire
-		(pts
-			(xy 254.92 100.0) (xy 247.3 100.0)
-		)
-		(stroke
-			(width 0)
-			(type default)
-		)
-	)
-	(label "GATE_SIGNAL"
-		(at 247.3 100.0 0)
-		(effects
-			(font
-				(size 1.27 1.27)
-			)
-			(justify right bottom)
-		)
-	)
-	(wire
-		(pts
-			(xy 262.54 94.92) (xy 262.54 84.76)
-		)
-		(stroke
-			(width 0)
-			(type default)
-		)
-	)
-	(label "FET_DRAIN"
-		(at 262.54 84.76 90)
-		(effects
-			(font
-				(size 1.27 1.27)
-			)
-			(justify left bottom)
-		)
-	)
-	(wire
-		(pts
-			(xy 262.54 105.08) (xy 262.54 115.24)
-		)
-		(stroke
-			(width 0)
-			(type default)
-		)
-	)
-	(label "GND"
-		(at 262.54 115.24 90)
-		(effects
-			(font
-				(size 1.27 1.27)
-			)
-			(justify right bottom)
-		)
-	)
