File: ChipChat_Project/generated/Main_Amplifier_Circuit/Main_Amplifier_Circuit.kicad_sch (KiCad schematic)
At the start: 6 parts, among them J1 Connector_Generic:Conn_01x02, J2 Connector_Generic:Conn_01x02, U1 MCP6001

Commit message: 💾 snapshot 2026-03-21_19-51-56
Parts:
- removed U1: MCP6001, symbol MCP6001R
- added C2, C3: 0.1uF, symbol Capacitor
- added J3: Connector_Generic:Conn_01x02, symbol Conn_01x02
- added U1: OpAmp_Single, symbol LM741
- C1: value 0.1uF -> 10uF
- R2: value 10K -> 20K
Connections:
- net GND: now also R1.1, C2.1, C3.1, J3.2 (Pin_2), U1.4 (V-); no longer R2.1
- net Vin renamed PWR_15V
- net PWR_15V: now also C2.2, C3.2, U1.7 (V+); no longer R1.2
- net Vin_Half renamed J_OUT_SIG
- net J_OUT_SIG: now also J3.1 (Pin_1), U1.6; no longer R1.1
- net Vout renamed J_IN_SIG
- net J_IN_SIG: now also U1.3 (+)
- new net U1_IN_MINUS: R1.2, R2.1, U1.2 (-)
