File: ChipChat_Project/generated/nRF5340_BaseBoard/nRF5340_Core.kicad_sch (KiCad schematic)
At the start: 10 parts, among them U1 nRF5340_SoC, X1 Device:Crystal

Commit message: 💾 snapshot 2026-03-23_13-16-53
Connections:
- net RESET_N_MCU: now also U1.AC31 (~{RESET})
- net U1_XL1: now also U1.N1 (XL1/P0.00)
- net U1_XL2: now also U1.R1 (XL2/P0.01)
- net VCC_3V3: no longer U1.E1 (VDDH), U1.V2 (AIN0/P0.04)
- net SWDIO_MCU: now reaches U1.AA31 (SWDIO)
- net SWDCLK_MCU: now reaches U1.W31 (SWDCLK)
Changed lines of the file:
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@@
-	(wire
-		(pts
-			(xy 213.02 44.12) (xy 220.64 44.12)
-		)
-		(stroke
-			(width 0)
-			(type default)
-		)
-	)
-	(label "VCC_3V3"
-		(at 220.64 44.12 0)
-		(effects
-			(font
-				(size 1.27 1.27)
-			)
-			(justify left bottom)
-		)
-	)
-	(wire
-		(pts
-			(xy 180.0 26.34) (xy 180.0 16.18)
-		)
-		(stroke
-			(width 0)
-			(type default)
-		)
-	)
-	(label "VCC_3V3"
-		(at 180.0 16.18 90)
-		(effects
-			(font
-				(size 1.27 1.27)
-			)
-			(justify left bottom)
-		)
-	)
 	(wire
 		(pts
@@
 		)
 	)
+	(wire
+		(pts
+			(xy 213.02 33.96) (xy 220.64 33.96)
+		)
+		(stroke
+			(width 0)
+			(type default)
+		)
+	)
+	(label "U1_XL1"
+		(at 220.64 33.96 0)
+		(effects
+			(font
+				(size 1.27 1.27)
+			)
+			(justify left bottom)
+		)
+	)
+	(wire
+		(pts
+			(xy 213.02 36.5) (xy 220.64 36.5)
+		)
+		(stroke
+			(width 0)
+			(type default)
+		)
+	)
+	(label "U1_XL2"
+		(at 220.64 36.5 0)
+		(effects
+			(font
+				(size 1.27 1.27)
+			)
+			(justify left bottom)
+		)
+	)
+	(wire
+		(pts
+			(xy 146.98 36.5) (xy 139.36 36.5)
+		)
+		(stroke
+			(width 0)
+			(type default)
+		)
+	)
+	(hierarchical_label "SWDIO_MCU"
+		(shape bidirectional)
+		(at 139.36 36.5 180)
+		(effects
+			(font
+				(size 1.27 1.27)
+			)
+			(justify right)
+		)
+	)
+	(wire
+		(pts
+			(xy 146.98 33.96) (xy 139.36 33.96)
+		)
+		(stroke
+			(width 0)
+			(type default)
+		)
+	)
+	(hierarchical_label "SWDCLK_MCU"
+		(shape bidirectional)
+		(at 139.36 33.96 180)
+		(effects
+			(font
+				(size 1.27 1.27)
+			)
+			(justify right)
+		)
+	)
+	(wire
+		(pts
+			(xy 146.98 39.04) (xy 139.36 39.04)
+		)
+		(stroke
+			(width 0)
+			(type default)
+		)
+	)
+	(hierarchical_label "RESET_N_MCU"
+		(shape bidirectional)
+		(at 139.36 39.04 180)
+		(effects
+			(font
+				(size 1.27 1.27)
+			)
+			(justify right)
+		)
+	)
