File: Code/generated/BME280_Sensor.kicad_sch (KiCad schematic)
At the start: 8 parts, among them U3 BME280

Commit message: stable release in kicad10-cursor- april 29 follow-up: everything working before making this a server online
Made-with: Cursor
Parts:
- removed C10, C9: 0.1uF, symbol Capacitor
- removed R5, R6: 4.7K, symbol Resistor
- removed R7, R8, R9: 0R, symbol Resistor
- removed U3: BME280, symbol BME280
- added C10, C9: 0.1uF, Capacitor_SMD:C_0603_1608Metric, symbol SchematIQ:Capacitor
- added R5, R6: 4.7K, Resistor_SMD:R_0603_1608Metric, symbol SchematIQ:Resistor
- added R7, R8, R9: 0R, Resistor_SMD:R_0603_1608Metric, symbol SchematIQ:Resistor
- added U3: BME280, BME280:PSON65P250X250X100-8N, symbol SchematIQ:BME280
Connections:
- net GND: now also C10.1, C9.1, R9.1, U3.1 (GND), U3.7 (GND)
- net I2C_SCL_0R: now also R7.1, U3.4 (SCK)
- net I2C_SCL_BME: now also R5.2, R7.2
- net I2C_SDA_0R: now also R8.1, U3.3 (SDI)
- net I2C_SDA_BME: now also R6.2, R8.2
- net PP_3V3_OUT: now also C10.2, C9.2, R5.1, R6.1, U3.6 (VDDIO), U3.8 (VDD)
- net SDO_ADD: now also R9.2, U3.5 (SDO)
