File: Code/generated/Buck_Converter.kicad_sch (KiCad schematic)
At the start: 6 parts, among them U1 TPS628438DRL

Commit message: stable release in kicad10-cursor- april 29 follow-up: everything working before making this a server online
Made-with: Cursor
Parts:
- removed C3, C5: 4.7uF, symbol Capacitor
- removed C4: 0.1uF, symbol Capacitor
- removed L1: 1.0uH, symbol L
- removed R3: 249K, symbol Resistor
- removed U1: TPS628438DRL, symbol TPS628436DRL
- added C3, C5: 4.7uF, Capacitor_SMD:C_0603_1608Metric, symbol SchematIQ:Capacitor
- added C4: 0.1uF, Capacitor_SMD:C_0603_1608Metric, symbol SchematIQ:Capacitor
- added L1: 1.0uH, Inductor_SMD:L_0603_1608Metric, symbol SchematIQ:L
- added R3: 249K, Resistor_SMD:R_0603_1608Metric, symbol SchematIQ:Resistor
- added U1: TPS628438DRL, Package_TO_SOT_SMD:SOT-563, symbol SchematIQ:TPS628436DRL
Connections:
- net BUCK_SW: now also L1.2, U1.5 (SW)
- net Buck_Vset_3V3: now also R3.2, U1.3 (VSET)
- net GND: now also C3.1, C4.1, C5.1, R3.1, U1.1 (GND)
- net PP_3V3_OUT: now also C5.2, L1.1, U1.6 (VOS)
- net PP_5V_SYS: now also C3.2, C4.2, U1.2 (VIN), U1.4 (EN)
