File: Code/generated/USBC.kicad_sch (KiCad schematic)
At the start: 11 parts, among them J1 USB_C_Receptacle_USB2.0_16P

Commit message: stable release in kicad10-cursor- april 29 follow-up: everything working before making this a server online
Made-with: Cursor
Parts:
- removed C1: 0.1uF, symbol Capacitor
- removed C2: 4.7uF, symbol Capacitor
- removed D1, D2, D3, D4, D5: TVS 5V, symbol SD05_SOD323
- removed FB1: 120Ω@100MHz, symbol FerriteBead
- removed J1: USB_C_Receptacle_USB2.0_16P, symbol USB_C_Receptacle_USB2.0_16P
- removed R1, R2: 5.1K, symbol Resistor
- added C1: 0.1uF, Capacitor_SMD:C_0603_1608Metric, symbol SchematIQ:Capacitor
- added C2: 4.7uF, Capacitor_SMD:C_0603_1608Metric, symbol SchematIQ:Capacitor
- added D1, D2, D3, D4, D5: TVS 5V, Diode_SMD:D_SOD-323, symbol SchematIQ:SD05_SOD323
- added FB1: 120Ω@100MHz, Inductor_SMD:L_0603_1608Metric, symbol SchematIQ:FerriteBead
- added J1: USB_C_Receptacle_USB2.0_16P, symbol SchematIQ:USB_C_Receptacle_USB2.0_16P
- added R1, R2: 5.1K, Resistor_SMD:R_0603_1608Metric, symbol SchematIQ:Resistor
Connections:
- net GND: now also C1.1, C2.1, D1.2 (A2), D2.2 (A2), D3.2 (A2), D4.2 (A2), D5.2 (A2), J1.A1 (GND), J1.A12 (GND), J1.B1 (GND), J1.B12 (GND), J1.S1 (SHIELD), R1.1, R2.1
- net PP_5V_SYS: now also FB1.1
- net PP_5V_VBUS: now also C1.2, C2.2, D5.1 (A1), FB1.2, J1.A4 (VBUS), J1.A9 (VBUS), J1.B4 (VBUS), J1.B9 (VBUS)
- net USB_CC1: now also D4.1 (A1), J1.A5 (CC1), R1.2
- net USB_CC2: now also J1.B5 (CC2), R2.2
- net USB_DN: now also D1.1 (A1), D2.1 (A1), J1.A7 (D-), J1.B7 (D-)
- net USB_DP: now also D3.1 (A1), J1.A6 (D+), J1.B6 (D+)
