File: Code/generated/USB_To_I2C.kicad_sch (KiCad schematic)
At the start: 5 parts, among them U2 MCP2221A-I_SL

Commit message: stable release in kicad10-cursor- april 29 follow-up: everything working before making this a server online
Made-with: Cursor
Parts:
- removed C6: 0.47uF, symbol Capacitor
- removed C7: 0.1uF, symbol Capacitor
- removed C8: 1uF, symbol Capacitor
- removed R4: 10K, symbol Resistor
- removed U2: MCP2221A-I_SL, symbol MCP2221A-I_SL
- added C6: 0.47uF, Capacitor_SMD:C_0603_1608Metric, symbol SchematIQ:Capacitor
- added C7: 0.1uF, Capacitor_SMD:C_0603_1608Metric, symbol SchematIQ:Capacitor
- added C8: 1uF, Capacitor_SMD:C_0603_1608Metric, symbol SchematIQ:Capacitor
- added R4: 10K, Resistor_SMD:R_0603_1608Metric, symbol SchematIQ:Resistor
- added U2: MCP2221A-I_SL, MCP2221A-I_SL:SOIC127P600X175-14N, symbol SchematIQ:MCP2221A-I_SL
Connections:
- net GND: now also C6.1, C7.1, C8.1, U2.14 (VSS)
- net I2C_SCL_BME: now also U2.10 (SCL)
- net I2C_SDA_BME: now also U2.9 (SDA)
- net MCP_NRST: now also R4.2, U2.4 (~{RST})
- net PP_3V3_OUT: now also C7.2, C8.2, R4.1, U2.1 (VDD)
- net PP_5V_SYS: now also C6.2
- net USB_DN: now also U2.12 (D-)
- net USB_DP: now also U2.13 (D+)
